Commit message: Fix colors for Gazebo

File: description/robot_core.xacro (robot description, xacro)
@@ -48,4 +48,8 @@
         </xacro:inertial_box>
     </link>
+    <!-- Assign color in Gazebo -->
+    <gazebo reference="chassis">
+        <material>Gazebo/White</material>
+    </gazebo>
     <!-- Left wheel joint -->
     <joint name="left_wheel_joint" type="continuous">
@@ -73,4 +77,8 @@
         </xacro:inertial_cylinder>
     </link>
+    <!-- Assign color in Gazebo -->
+    <gazebo reference="left_wheel">
+        <material>Gazebo/Blue</material>
+    </gazebo>
     <!-- Right wheel joint -->
     <joint name="right_wheel_joint" type="continuous">
@@ -97,4 +105,8 @@
         </xacro:inertial_cylinder>
     </link>
+    <!-- Assign color in Gazebo -->
+    <gazebo reference="right_wheel">
+        <material>Gazebo/Blue</material>
+    </gazebo>
     <!-- Caster wheel joint -->
     <joint name="caster_wheel_joint" type="fixed">
@@ -120,3 +132,7 @@
         </xacro:inertial_sphere>
     </link>
+    <!-- Assign color in Gazebo -->
+    <gazebo reference="caster_wheel">
+        <material>Gazebo/Black</material>
+    </gazebo>
 </robot>
