Commit message: Add depth camera sensor, Update rviz config

File: description/camera.xacro (robot description, xacro)
@@ -27,5 +27,5 @@
         <sensor name="camera" type="camera">
             <pose> 0 0 0 0 0 0 </pose>
-            <visualize> true </visualize>
+            <visualize> false </visualize>
             <update_rate> 10</update_rate>
             <camera>

File: description/robot.urdf.xacro (robot description, xacro)
@@ -5,3 +5,4 @@
     <xacro:include filename="lidar.xacro" />
     <xacro:include filename="camera.xacro" />
+    <xacro:include filename="depth_camera.xacro" />
 </robot>

File: description/robot_core.xacro (robot description, xacro)
@@ -18,4 +18,7 @@
     <material name="red">
         <color rgba="1 0 0 1"/>
+    </material>
+    <material name="green">
+        <color rgba="0 1 0 1"/>
     </material>
     <!-- Initialize the base link -->

Commit message: New robot skin added

File: description/camera.xacro (robot description, xacro)
@@ -1,19 +1,61 @@
 <?xml version="1.0"?>
 <robot xmlns:xacro="http://www.ros.org/wiki/xacro">
-    <!-- Camera joint and link  -->
-    <joint name="camera_joint" type="fixed">
+    <!-- Define camera colors -->
+    <material name="camera_black">
+        <color rgba="0.1 0.1 0.1 1"/>
+    </material>
+    <material name="camera_lens_blue">
+        <color rgba="0.2 0.3 0.8 1"/>
+    </material>
+    <!-- Camera positioned higher and further forward -->
+    <joint name="camera_body_joint" type="fixed">
         <parent link="chassis"/>
-        <child link="camera_link"/>
-        <origin xyz="0.305 0 0.1" rpy="0 0 0"/>
+        <child link="camera_body"/>
+        <origin xyz="0.31 0 0.1" rpy="0 0.05 0"/>  <!-- Moved up to 0.12, forward to 0.31, slight downward tilt -->
     </joint>
-    <link name="camera_link">
+    <link name="camera_body">
         <visual>
             <geometry>
-                <box size="0.015 0.03 0.03"/>
+                <box size="0.02 0.03 0.03"/>
             </geometry>
-            <material name="orange"/>
+            <material name="camera_black"/>
+        </visual>
+        <collision>
+            <geometry>
+                <box size="0.02 0.03 0.03"/>
+            </geometry>
+        </collision>
+        <xacro:inertial_box mass="0.02" x="0.02" y="0.03" z="0.03">
+            <origin xyz="0 0 0" rpy="0 0 0"/>
+        </xacro:inertial_box>
+    </link>
+    <gazebo reference="camera_body">
+        <material>Gazebo/Black</material>
+    </gazebo>
+    <!-- Lens indicator -->
+    <joint name="camera_lens_visual_joint" type="fixed">
+        <parent link="camera_body"/>
+        <child link="camera_lens_visual"/>
+        <origin xyz="0.011 0 0" rpy="0 1.5708 0"/>
+    </joint>
+    <link name="camera_lens_visual">
+        <visual>
+            <geometry>
+                <cylinder radius="0.005" length="0.002"/>
+            </geometry>
+            <material name="camera_lens_blue"/>
         </visual>
     </link>
-    <!-- Camera joint and link optical for different frame of reference -->
+    <gazebo reference="camera_lens_visual">
+        <material>Gazebo/Blue</material>
+    </gazebo>
+    <!-- Camera sensor link -->
+    <joint name="camera_joint" type="fixed">
+        <parent link="camera_body"/>
+        <child link="camera_link"/>
+        <origin xyz="0.02 0 0" rpy="0 0 0"/>  <!-- Well in front of body -->
+    </joint>
+    <link name="camera_link"/>
+    <!-- Camera optical frame -->
     <joint name="camera_joint_optical" type="fixed">
         <parent link="camera_link"/>
@@ -21,14 +63,14 @@
         <origin xyz="0 0 0" rpy="${-pi/2} 0 ${-pi/2}"/>
     </joint>
-    <link name="camera_link_optical"></link>
-    <!-- Gazebo reference for camera_link -->
+    <link name="camera_link_optical"/>
+    <!-- Gazebo sensor with adjusted FOV -->
     <gazebo reference="camera_link">
-        <material>Gazebo/Orange</material>
         <sensor name="camera" type="camera">
-            <pose> 0 0 0 0 0 0 </pose>
-            <visualize> false </visualize>
-            <update_rate> 10</update_rate>
+            <pose>0 0 0 0 0 0</pose>
+            <always_on>true</always_on>
+            <visualize>true</visualize>  <!-- Enable to see camera frustum -->
+            <update_rate>30</update_rate>
             <camera>
-                <horizontal_fov>1.089</horizontal_fov>
+                <horizontal_fov>1.396</horizontal_fov>  <!-- Wider FOV ~80 degrees -->
                 <image>
                     <format>R8G8B8</format>
@@ -37,9 +79,15 @@
                 </image>
                 <clip>
-                    <near>0.05</near>
-                    <far>8.0</far>
+                    <near>0.05</near>  <!-- Increased to avoid seeing nearby objects -->
+                    <far>100.0</far>
                 </clip>
             </camera>
             <plugin name="camera_controller" filename="libgazebo_ros_camera.so">
+                <ros>
+                    <namespace>/</namespace>
+                    <remapping>image_raw:=camera/image_raw</remapping>
+                    <remapping>camera_info:=camera/camera_info</remapping>
+                </ros>
+                <camera_name>camera</camera_name>
                 <frame_name>camera_link_optical</frame_name>
             </plugin>

File: description/depth_camera.xacro (robot description, xacro)
@@ -1,19 +1,114 @@
 <?xml version="1.0"?>
 <robot xmlns:xacro="http://www.ros.org/wiki/xacro">
-    <!-- Depth camera joint and link  -->
+    <!-- Define depth camera colors -->
+    <material name="depth_camera_black">
+        <color rgba="0.05 0.05 0.05 1"/>
+    </material>
+    <material name="depth_camera_dark_grey">
+        <color rgba="0.3 0.3 0.3 1"/>
+    </material>
+    <!-- Depth camera housing -->
+    <joint name="depth_camera_housing_joint" type="fixed">
+        <parent link="chassis"/>
+        <child link="depth_camera_housing"/>
+        <origin xyz="0.295 0 0.13" rpy="0 0 0"/>
+    </joint>
+    <link name="depth_camera_housing">
+        <visual>
+            <geometry>
+                <box size="0.02 0.095 0.02"/>
+            </geometry>
+            <material name="depth_camera_black"/>
+        </visual>
+        <collision>
+            <geometry>
+                <box size="0.02 0.095 0.02"/>
+            </geometry>
+        </collision>
+        <xacro:inertial_box mass="0.03" x="0.02" y="0.095" z="0.02">
+            <origin xyz="0 0 0" rpy="0 0 0"/>
+        </xacro:inertial_box>
+    </link>
+    <gazebo reference="depth_camera_housing">
+        <material>Gazebo/Black</material>
+    </gazebo>
+    <!-- Left IR camera -->
+    <joint name="depth_left_ir_joint" type="fixed">
+        <parent link="depth_camera_housing"/>
+        <child link="depth_left_ir"/>
+        <origin xyz="0.011 0.035 0" rpy="0 1.5708 0"/>
+    </joint>
+    <link name="depth_left_ir">
+        <visual>
+            <geometry>
+                <cylinder radius="0.005" length="0.003"/>
+            </geometry>
+            <material name="depth_camera_dark_grey"/>
+        </visual>
+    </link>
+    <gazebo reference="depth_left_ir">
+        <material>Gazebo/DarkGrey</material>
+    </gazebo>
+    <!-- Right IR camera -->
+    <joint name="depth_right_ir_joint" type="fixed">
+        <parent link="depth_camera_housing"/>
+        <child link="depth_right_ir"/>
+        <origin xyz="0.011 -0.035 0" rpy="0 1.5708 0"/>
+    </joint>
+    <link name="depth_right_ir">
+        <visual>
+            <geometry>
+                <cylinder radius="0.005" length="0.003"/>
+            </geometry>
+            <material name="depth_camera_dark_grey"/>
+        </visual>
+    </link>
+    <gazebo reference="depth_right_ir">
+        <material>Gazebo/DarkGrey</material>
+    </gazebo>
+    <!-- RGB camera in center -->
+    <joint name="depth_rgb_joint" type="fixed">
+        <parent link="depth_camera_housing"/>
+        <child link="depth_rgb"/>
+        <origin xyz="0.011 0 0" rpy="0 1.5708 0"/>
+    </joint>
+    <link name="depth_rgb">
+        <visual>
+            <geometry>
+                <cylinder radius="0.004" length="0.003"/>
+            </geometry>
+            <material name="depth_camera_dark_grey"/>
+        </visual>
+    </link>
+    <gazebo reference="depth_rgb">
+        <material>Gazebo/DarkGrey</material>
+    </gazebo>
+    <!-- IR projector (between left camera and RGB) -->
+    <joint name="depth_projector_joint" type="fixed">
+        <parent link="depth_camera_housing"/>
+        <child link="depth_projector"/>
+        <origin xyz="0.011 0.0175 0" rpy="0 1.5708 0"/>
+    </joint>
+    <link name="depth_projector">
+        <visual>
+            <geometry>
+                <cylinder radius="0.003" length="0.003"/>
+            </geometry>
+            <material name="red"/>
+        </visual>
+    </link>
+    <gazebo reference="depth_projector">
+        <material>Gazebo/RedGlow</material>
+    </gazebo>
+    <!-- Main depth camera link (hidden, for sensor attachment) -->
     <joint name="depth_camera_joint" type="fixed">
-        <parent link="chassis"/>
+        <parent link="depth_camera_housing"/>
         <child link="depth_camera_link"/>
-        <origin xyz="0.305 0 0.13" rpy="0 0 0"/>
+        <origin xyz="0.01 0 0" rpy="0 0 0"/>
     </joint>
     <link name="depth_camera_link">
-        <visual>
-            <geometry>
-                <box size="0.015 0.09 0.015"/>
-            </geometry>
-            <material name="green"/>
-        </visual>
+        <!-- No visual, just for sensor attachment -->
     </link>
-    <!-- Depth camera joint and link optical for different frame of reference -->
+    <!-- Depth camera optical frame -->
     <joint name="depth_camera_joint_optical" type="fixed">
         <parent link="depth_camera_link"/>
@@ -22,11 +117,10 @@
     </joint>
     <link name="depth_camera_link_optical"></link>
-    <!-- Gazebo reference for depth_camera_link -->
+    <!-- Gazebo sensor configuration -->
     <gazebo reference="depth_camera_link">
-        <material>Gazebo/Green</material>
-        <sensor name="camera" type="depth">
+        <sensor name="depth_camera" type="depth">
             <pose> 0 0 0 0 0 0 </pose>
-            <visualize> true </visualize>
-            <update_rate> 10</update_rate>
+            <visualize>false</visualize>
+            <update_rate>10</update_rate>
             <camera>
                 <horizontal_fov>1.089</horizontal_fov>

File: description/lidar.xacro (robot description, xacro)
@@ -1,8 +1,41 @@
 <?xml version="1.0"?>
 <robot xmlns:xacro="http://www.ros.org/wiki/xacro">
+    <!-- Define lidar-specific colors -->
+    <material name="lidar_black">
+        <color rgba="0.1 0.1 0.1 1"/>
+    </material>
+    <material name="lidar_white">
+        <color rgba="1 1 1 1"/>
+    </material>
+    <!-- Lidar base mount -->
+    <joint name="lidar_base_joint" type="fixed">
+        <parent link="chassis"/>
+        <child link="lidar_base"/>
+        <origin xyz="0.1 0 0.15" rpy="0 0 0"/>
+    </joint>
+    <link name="lidar_base">
+        <visual>
+            <geometry>
+                <cylinder radius="0.04" length="0.015"/>
+            </geometry>
+            <material name="lidar_black"/>
+        </visual>
+        <collision>
+            <geometry>
+                <cylinder radius="0.04" length="0.015"/>
+            </geometry>
+        </collision>
+        <xacro:inertial_cylinder mass="0.02" radius="0.04" length="0.015">
+            <origin xyz="0 0 0" rpy="0 0 0"/>
+        </xacro:inertial_cylinder>
+    </link>
+    <gazebo reference="lidar_base">
+        <material>Gazebo/Black</material>
+    </gazebo>
+    <!-- Main lidar sensor (laser_frame for compatibility) -->
     <joint name="laser_joint" type="fixed">
-        <parent link="chassis"/>
+        <parent link="lidar_base"/>
         <child link="laser_frame"/>
-        <origin xyz="0.1 0 0.155" rpy="0 0 0"/>
+        <origin xyz="0 0 0.0125" rpy="0 0 0"/>
     </joint>
     <link name="laser_frame">
@@ -11,5 +44,5 @@
                 <cylinder radius="0.035" length="0.02"/>
             </geometry>
-            <material name="red"/>
+            <material name="lidar_white"/>
         </visual>
         <collision>
@@ -18,34 +51,70 @@
             </geometry>
         </collision>
-        <xacro:inertial_cylinder mass="0.05" radius="0.025" length="0.02">
+        <xacro:inertial_cylinder mass="0.05" radius="0.035" length="0.02">
             <origin xyz="0 0 0" rpy="0 0 0"/>
         </xacro:inertial_cylinder>
     </link>
+    <!-- Lidar lens ring (transparent part) -->
+    <joint name="lidar_lens_joint" type="fixed">
+        <parent link="laser_frame"/>
+        <child link="lidar_lens"/>
+        <origin xyz="0 0 0" rpy="0 0 0"/>
+    </joint>
+    <link name="lidar_lens">
+        <visual>
+            <geometry>
+                <cylinder radius="0.037" length="0.015"/>
+            </geometry>
+            <material name="lidar_black"/>
+        </visual>
+    </link>
+    <gazebo reference="lidar_lens">
+        <material>Gazebo/GreyTransparent</material>
+    </gazebo>
+    <!-- Top detail -->
+    <joint name="lidar_top_joint" type="fixed">
+        <parent link="laser_frame"/>
+        <child link="lidar_top"/>
+        <origin xyz="0 0 0.011" rpy="0 0 0"/>
+    </joint>
+    <link name="lidar_top">
+        <visual>
+            <geometry>
+                <cylinder radius="0.025" length="0.002"/>
+            </geometry>
+            <material name="lidar_black"/>
+        </visual>
+    </link>
+    <gazebo reference="lidar_top">
+        <material>Gazebo/Black</material>
+    </gazebo>
+    <!-- Gazebo sensor configuration -->
     <gazebo reference="laser_frame">
-        <material>Gazebo/Red</material>
+        <material>Gazebo/DarkGrey</material>
         <sensor name="laser" type="ray">
             <pose> 0 0 0 0 0 0 </pose>
-            <visualize> false </visualize>
-            <update_rate> 10</update_rate>
+            <visualize>false</visualize>
+            <update_rate>10</update_rate>
             <ray>
                 <scan>
                     <horizontal>
-                        <samples>360</samples>          <!--Number of samples per scan-->
+                        <samples>360</samples>
                         <resolution>1</resolution>
-                        <min_angle>-3.14</min_angle>    <!--Min angle -pi-->
-                        <max_angle>3.14</max_angle>     <!--Max angle pi-->
+                        <min_angle>-3.14</min_angle>
+                        <max_angle>3.14</max_angle>
                     </horizontal>
                 </scan>
                 <range>
-                    <min>0.3</min>                      <!--Min range-->
-                    <max>12</max>                       <!--Max range-->
+                    <min>0.3</min>
+                    <max>12</max>
                 </range>
             </ray>
             <plugin name="laser_controller" filename="libgazebo_ros_ray_sensor.so">
                 <ros>
-                    <argument>~/out:=lidar_scan</argument>    <!--Topic name-->
+                    <namespace>/</namespace>
+                    <remapping>~/out:=lidar_scan</remapping>
                 </ros>
-                <output_type>sensor_msgs/LaserScan</output_type>    <!--ros message service for Lidar-->
-                <frame_name>Laser Frame</frame_name>
+                <output_type>sensor_msgs/LaserScan</output_type>
+                <frame_name>laser_frame</frame_name>
             </plugin>
         </sensor>

File: description/robot_core.xacro (robot description, xacro)
@@ -22,4 +22,10 @@
         <color rgba="0 1 0 1"/>
     </material>
+    <material name="wheel_color">
+        <color rgba="0.1 0.1 0.1 1"/> <!-- Dark grey -->
+    </material>
+    <material name="chassis_color">
+        <color rgba="0.8 0.4 0.1 1.0"/>  <!-- Darker orange -->
+    </material>
     <!-- Initialize the base link -->
     <link name="base_link">
@@ -39,5 +45,5 @@
                 <box size="0.3 0.3 0.15"/> <!-- Size of the robot in meters -->
             </geometry>
-            <material name="white"/>
+            <material name="chassis_color"/>
         </visual>
         <collision>
@@ -56,5 +62,12 @@
     <!-- Assign color in Gazebo -->
     <gazebo reference="chassis">
-        <material>Gazebo/White</material>
+        <visual>
+            <material>
+                <ambient>0.5 0.2 0.05 1.0</ambient>
+                <diffuse>0.7 0.3 0.1 1.0</diffuse>
+                <specular>0.8 0.8 0.8 1.0</specular>
+                <emissive>0.0 0.0 0.0 0.0</emissive>
+            </material>
+        </visual>
     </gazebo>
     <!-- Left wheel joint -->
@@ -71,9 +84,9 @@
                 <cylinder radius="0.05" length="0.04"/>
             </geometry>
-            <material name="blue"/>
+            <material name="wheel_color"/>
         </visual>
         <collision>
             <geometry>
-                <cylinder radius="0.05" length="0.04"/>
+                <sphere radius="0.05"/>
             </geometry>
         </collision>
@@ -85,5 +98,5 @@
     <!-- Assign color in Gazebo -->
     <gazebo reference="left_wheel">
-        <material>Gazebo/Blue</material>
+        <material>Gazebo/FlatBlack</material>
     </gazebo>
     <!-- Right wheel joint -->
@@ -100,9 +113,9 @@
                 <cylinder radius="0.05" length="0.04"/>
             </geometry>
-            <material name="blue"/>
+            <material name="wheel_color"/>
         </visual>
         <collision>
             <geometry>
-                <cylinder radius="0.05" length="0.04"/>
+                <sphere radius="0.05"/>
             </geometry>
         </collision>
@@ -113,5 +126,5 @@
     <!-- Assign color in Gazebo -->
     <gazebo reference="right_wheel">
-        <material>Gazebo/Blue</material>
+        <material>Gazebo/FlatBlack</material>
     </gazebo>
     <!-- Caster wheel joint -->
@@ -127,5 +140,5 @@
                 <sphere radius="0.05"/>
             </geometry>
-            <material name="black"/>
+            <material name="wheel_color"/>
         </visual>
         <collision>
@@ -138,8 +151,6 @@
         </xacro:inertial_sphere>
     </link>
-    <!-- Assign color in Gazebo -->
     <gazebo reference="caster_wheel">
-        <material>Gazebo/Black</material>
-        <!-- Remove friction for caster wheel -->
+        <material>Gazebo/DarkGrey</material>
         <mu1>0.001</mu1>
         <mu2>0.001</mu2>
