Commit message: Bug fixes in xacro, updated world and rviz config

File: description/lidar.xacro (robot description, xacro)
@@ -112,6 +112,5 @@
             <plugin name="laser_controller" filename="libgazebo_ros_ray_sensor.so">
                 <ros>
-                    <namespace>/</namespace>
-                    <remapping>~/out:=lidar_scan</remapping>
+                    <argument>~/out:=scan</argument>
                 </ros>
                 <output_type>sensor_msgs/LaserScan</output_type>

File: description/robot_core.xacro (robot description, xacro)
@@ -31,4 +31,11 @@
     <link name="base_link">
     </link>
+    <!-- Base footprint joint and link -->
+    <joint name="base_footprint_joint" type="fixed">
+        <parent link="base_link"/>
+        <child link="base_footprint"/>
+        <origin xyz="0 0 0" rpy="0 0 0"/>
+    </joint>
+    <link name="base_footprint"></link>
     <!-- Chassis joint -->
     <joint name="chassis_joint" type="fixed">
